File: SPROJ3G2_Controller_PCB.kicad_sch (KiCad schematic)
At the start: 65 parts, among them J1 SWDIO Con, J2 BMS Con, J3 2137160001, J4 OLED Con, J5 RF_Con, Q1 ZXMN3A03E6TA, Q2 ZXMN3A03E6TA, SW1 MTS-102, U1 W25Q128JVSIQ, U2 AMS1117-3.3, U3 RP2040, X1 ABM8-272-T3

Commit message: Schematic cleanup
Schematic cleanup
Other:
- note added: "12MHz Crystal Oscillator"
- note added: "2MB SPI Flash"
- note added: "BMS/Power connector"
- note added: "Boot button"
- note added: "SSD1306 128x32 I2C OLED display connector"
- note added: "Thumbsticks"
- note added: "nRF24L01 connector"
- note removed: "12MHz External Crystal Oscillator"
- note removed: "16MB SPI Flash EEPROM chip"
- note removed: "BMS Input Power- UART Connector"
- note removed: "Boot mode button"
- note removed: "Joysticks"
- note removed: "Pins for the SSD1306 128x32 I2C OLED Display"
- note removed: "Pins for the nRF24L01 communication module"
- company: SDU Sonderborg -> SDU Sønderborg
- title: SPROJ3G2 - Controller Logic PCB -> SPROJ3EEG2 - PTX PCB
Changed lines of the file:
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@@
 	(paper "A4")
 	(title_block
-		(title "SPROJ3G2 - Controller Logic PCB")
-		(date "2024-11-11")
-		(rev "1.4")
-		(company "SDU Sonderborg")
-		(comment 1 "Author: Bence Toth")
+		(title "SPROJ3EEG2 - PTX PCB")
+		(date "2024-12-20")
+		(rev "1.6")
+		(company "SDU Sønderborg")
+		(comment 1 "Author: Bence Tóth")
 	)
 	(junction
@@
 		)
 	)
-	(text "12MHz External Crystal Oscillator"
+	(text "12MHz Crystal Oscillator"
 		(exclude_from_sim no)
 		(at 146.812 69.85 0)
@@
 		)
 	)
-	(text "Pins for the nRF24L01\ncommunication module"
+	(text "nRF24L01 connector"
 		(exclude_from_sim no)
 		(at 112.776 98.298 0)
@@
 		)
 	)
-	(text "Pins for the SSD1306\n128x32 I2C OLED Display"
+	(text "SSD1306 128x32 I2C\nOLED display connector"
 		(exclude_from_sim no)
 		(at 62.23 103.632 0)
@@
 		)
 	)
-	(text "Boot mode button"
+	(text "Boot button"
 		(exclude_from_sim no)
 		(at 104.902 23.114 0)
@@
 	(text "USB-C 2.0 Port"
 		(exclude_from_sim no)
-		(at 152.4 177.292 0)
+		(at 162.56 128.27 0)
 		(effects
 			(font
@@
 		)
 	)
-	(text "Joysticks"
+	(text "Thumbsticks"
 		(exclude_from_sim no)
-		(at 70.104 68.326 0)
+		(at 70.866 66.294 0)
 		(effects
 			(font
@@
 		)
 	)
-	(text "16MB SPI Flash EEPROM chip"
+	(text "2MB SPI Flash"
 		(exclude_from_sim no)
 		(at 44.704 16.51 0)
@@
 	(text "Logic level shifters for\nthe BMS UART communication"
 		(exclude_from_sim no)
-		(at 62.738 165.1 0)
+		(at 59.436 165.1 0)
 		(effects
 			(font
@@
 	(text "3.3V Linear Voltage Regulator"
 		(exclude_from_sim no)
-		(at 90.17 133.604 0)
+		(at 87.63 133.604 0)
 		(effects
 			(font
@@
 		)
 	)
-	(text "BMS Input Power-\nUART Connector"
+	(text "BMS/Power connector"
 		(exclude_from_sim no)
-		(at 26.416 130.048 0)
+		(at 31.496 132.842 0)
 		(effects
 			(font
@@
 		(dnp no)
 		(property "Reference" "J3"
-			(at 146.05 129.032 0)
+			(at 146.05 176.276 0)
 			(effects
 				(font
