File: SPROJ3G2_Controller_PCB.kicad_pcb (KiCad board)
At the start: 2 copper layers, 100 x 60 mm, 69 parts, among them J1 SWDIO Con, J2 BMS Con, J3 2137160001, J4 OLED Con, J5 RF_Con, Q1 ZXMN3A03E6TA, Q2 ZXMN3A03E6TA, SW1 MTS-102, U1 W25Q128JVSIQ, U2 AMS1117-3.3, U3 RP2040, X1 ABM8-272-T3

Commit message: Clean-up
Clean-up
Changed lines of the file:
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@@
 		(tags "Switch")
 		(property "Reference" "S1"
-			(at -0.937 9.175 0)
+			(at -3.9625 10.575 0)
 			(layer "F.SilkS")
 			(effects
@@
 		)
 		(fp_text user "${REFERENCE}"
-			(at -0.937 9.175 0)
+			(at -3.9625 10.575 0)
 			(layer "F.Fab")
 			(effects
@@
 	)
 	(segment
-		(start 128.896036 81.75)
+		(start 129.298656 81.75)
 		(end 122.15 81.75)
 		(width 0.6)
@@
 	)
 	(segment
-		(start 132.743792 83.343792)
+		(start 132.459098 83.059098)
 		(end 135.056207 85.656207)
 		(width 0.6)
@@
 	)
 	(arc
-		(start 132.743792 83.343792)
-		(mid 130.978426 82.164213)
-		(end 128.896036 81.75)
+		(start 132.459098 83.059098)
+		(mid 131.009075 82.090224)
+		(end 129.298656 81.75)
 		(width 0.6)
 		(layer "F.Cu")
